File: Power.sch (KiCad schematic (older format))
At the start: 0 parts

Commit message: Created CurrentDriver, Relay, and PowerProtection modules
Parts:
- added C? (x2): C, ~, symbol C
- added F? (x4): FUSE, ~, symbol FUSE
- added L? (x2): INDUCTOR, ~, symbol INDUCTOR
- added P?: CONN_12X2, symbol CONN_12X2
- added R?: R, ~, symbol R
- added SW?: SWITCH_INV, ~, symbol SWITCH_INV
Connections:
- net labels added: +12P, +12V, +3.3V, +5V, -12P, -12V, GND
- wire segments 0 -> 39

Commit message: Current driver refactoring, LED module, Arduino
Parts:
- removed F? (x4): FUSE, ~, symbol FUSE
- added TH? (x4): THERMISTOR, ~, symbol THERMISTOR
Connections:
- net labels added: +12C
- wire segments 39 -> 40
Changed lines of the file:
@@
 $Descr A4 11693 8268
 encoding utf-8
-Sheet 5 9
+Sheet 4 9
 Title ""
 Date "9 feb 2014"
@@
 $EndComp
 $Comp
-L FUSE F?
-U 1 1 52F67E8A
-P 3750 1850
-F 0 "F?" H 3850 1900 40  0000 C CNN
-F 1 "FUSE" H 3650 1800 40  0000 C CNN
-F 2 "~" H 3750 1850 60  0000 C CNN
-F 3 "~" H 3750 1850 60  0000 C CNN
-	1    3750 1850
-	1    0    0    -1
-$EndComp
-$Comp
-L FUSE F?
-U 1 1 52F67E97
-P 4500 2050
-F 0 "F?" H 4600 2100 40  0000 C CNN
-F 1 "FUSE" H 4400 2000 40  0000 C CNN
-F 2 "~" H 4500 2050 60  0000 C CNN
-F 3 "~" H 4500 2050 60  0000 C CNN
-	1    4500 2050
-	1    0    0    -1
-$EndComp
-$Comp
-L FUSE F?
-U 1 1 52F67E9D
-P 5300 2250
-F 0 "F?" H 5400 2300 40  0000 C CNN
-F 1 "FUSE" H 5200 2200 40  0000 C CNN
-F 2 "~" H 5300 2250 60  0000 C CNN
-F 3 "~" H 5300 2250 60  0000 C CNN
-	1    5300 2250
-	1    0    0    -1
-$EndComp
-$Comp
-L FUSE F?
-U 1 1 52F67EA3
-P 6000 2450
-F 0 "F?" H 6100 2500 40  0000 C CNN
-F 1 "FUSE" H 5900 2400 40  0000 C CNN
-F 2 "~" H 6000 2450 60  0000 C CNN
-F 3 "~" H 6000 2450 60  0000 C CNN
-	1    6000 2450
-	1    0    0    -1
-$EndComp
-$Comp
 L SWITCH_INV SW?
 U 1 1 52F67EC9
@@
 Connection ~ 3450 2050
 Wire Wire Line
-	5050 2250 3300 2250
-Wire Wire Line
-	5750 2450 3300 2450
+	5500 2250 3300 2250
+Wire Wire Line
+	6200 2450 3300 2450
 Wire Wire Line
 	4000 1850 4300 1850
@@
 	5000 2050 4750 2050
 Wire Wire Line
-	5800 1550 5800 2250
-Wire Wire Line
-	5800 2250 5550 2250
-Wire Wire Line
-	6650 2450 6250 2450
+	6250 1550 6250 2250
+Wire Wire Line
+	6250 2250 6000 2250
+Wire Wire Line
+	7100 2450 6700 2450
 $Comp
 L +12P #PWR?
 U 1 1 52F68365
-P 5800 1550
-F 0 "#PWR?" H 5800 1520 30  0001 C CNN
-F 1 "+12P" H 5800 1650 30  0000 C CNN
-F 2 "" H 5800 1550 60  0000 C CNN
-F 3 "" H 5800 1550 60  0000 C CNN
-	1    5800 1550
+P 6250 1550
+F 0 "#PWR?" H 6250 1520 30  0001 C CNN
+F 1 "+12P" H 6250 1650 30  0000 C CNN
+F 2 "" H 6250 1550 60  0000 C CNN
+F 3 "" H 6250 1550 60  0000 C CNN
+	1    6250 1550
 	1    0    0    -1
 $EndComp
@@
 L -12P #PWR?
 U 1 1 52F68398
-P 6650 1550
-F 0 "#PWR?" H 6650 1680 20  0001 C CNN
-F 1 "-12P" H 6650 1650 30  0000 C CNN
-F 2 "" H 6650 1550 60  0000 C CNN
-F 3 "" H 6650 1550 60  0000 C CNN
-	1    6650 1550
-	1    0    0    -1
-$EndComp
-Wire Wire Line
-	6650 1550 6650 2450
+P 7100 1550
+F 0 "#PWR?" H 7100 1680 20  0001 C CNN
+F 1 "-12P" H 7100 1650 30  0000 C CNN
+F 2 "" H 7100 1550 60  0000 C CNN
+F 3 "" H 7100 1550 60  0000 C CNN
+	1    7100 1550
+	1    0    0    -1
+$EndComp
+Wire Wire Line
+	7100 1550 7100 2450
 Wire Wire Line
 	1600 1950 2500 1950
@@
 	10000 3450 10000 3700
 Connection ~ 9450 3450
+$Comp
+L +12C #PWR?
+U 1 1 52F7CE7C
+P 5350 1550
+F 0 "#PWR?" H 5350 1520 30  0001 C CNN
+F 1 "+12C" H 5350 1660 40  0000 C CNN
+F 2 "" H 5350 1550 60  0000 C CNN
+F 3 "" H 5350 1550 60  0000 C CNN
+	1    5350 1550
+	1    0    0    -1
+$EndComp
+Wire Wire Line
+	5350 1550 5350 2250
+Connection ~ 5350 2250
+$Comp
+L THERMISTOR TH?
+U 1 1 52F7D3F0
+P 3750 1850
+F 0 "TH?" V 3850 1900 50  0000 C CNN
+F 1 "THERMISTOR" V 3650 1850 50  0000 C CNN
+F 2 "~" H 3750 1850 60  0000 C CNN
+F 3 "~" H 3750 1850 60  0000 C CNN
+	1    3750 1850
+	0    -1   -1   0
+$EndComp
+$Comp
+L THERMISTOR TH?
+U 1 1 52F7D3FF
+P 4500 2050
+F 0 "TH?" V 4600 2100 50  0000 C CNN
+F 1 "THERMISTOR" V 4400 2050 50  0000 C CNN
+F 2 "~" H 4500 2050 60  0000 C CNN
+F 3 "~" H 4500 2050 60  0000 C CNN
+	1    4500 2050
+	0    -1   -1   0
+$EndComp
+$Comp
+L THERMISTOR TH?
+U 1 1 52F7D40E
+P 5750 2250
+F 0 "TH?" V 5850 2300 50  0000 C CNN
+F 1 "THERMISTOR" V 5650 2250 50  0000 C CNN
+F 2 "~" H 5750 2250 60  0000 C CNN
+F 3 "~" H 5750 2250 60  0000 C CNN
+	1    5750 2250
+	0    -1   -1   0
+$EndComp
+$Comp
+L THERMISTOR TH?
+U 1 1 52F7D41D
+P 6450 2450
+F 0 "TH?" V 6550 2500 50  0000 C CNN
+F 1 "THERMISTOR" V 6350 2450 50  0000 C CNN
+F 2 "~" H 6450 2450 60  0000 C CNN
+F 3 "~" H 6450 2450 60  0000 C CNN
+	1    6450 2450
+	0    -1   -1   0
+$EndComp
 $EndSCHEMATC

Commit message: Refactoring and Created key shortcuts
Parts:
- added C?: C, ~, symbol C
- added L?: INDUCTOR, ~, symbol INDUCTOR
Connections:
- net +12V: now also L?.2
- net +3.3V: no longer TH?.2
- net +5V: now also C?.1, L?.2; no longer TH?.2
- net GND: now also C?.2
- new net +3.3VP: TH?.2
- new net +5P: L?.1, TH?.2
Other:
- moved on the sheet: C?, L?
Changed lines of the file:
@@
 Sheet 4 9
 Title ""
-Date "9 feb 2014"
+Date "18 feb 2014"
 Rev ""
 Comp ""
@@
 $EndComp
 $Comp
-L +5V #PWR?
-U 1 1 52F67E6C
-P 5000 1550
-F 0 "#PWR?" H 5000 1640 20  0001 C CNN
-F 1 "+5V" H 5000 1640 30  0000 C CNN
-F 2 "" H 5000 1550 60  0000 C CNN
-F 3 "" H 5000 1550 60  0000 C CNN
-	1    5000 1550
-	1    0    0    -1
-$EndComp
-$Comp
-L +3.3V #PWR?
-U 1 1 52F67E7B
-P 4300 1550
-F 0 "#PWR?" H 4300 1510 30  0001 C CNN
-F 1 "+3.3V" H 4300 1660 30  0000 C CNN
-F 2 "" H 4300 1550 60  0000 C CNN
-F 3 "" H 4300 1550 60  0000 C CNN
-	1    4300 1550
-	1    0    0    -1
-$EndComp
-$Comp
 L SWITCH_INV SW?
 U 1 1 52F67EC9
@@
 L +12P #PWR?
 U 1 1 52F684CA
-P 8150 1800
-F 0 "#PWR?" H 8150 1770 30  0001 C CNN
-F 1 "+12P" H 8150 1900 30  0000 C CNN
-F 2 "" H 8150 1800 60  0000 C CNN
-F 3 "" H 8150 1800 60  0000 C CNN
-	1    8150 1800
+P 8250 2300
+F 0 "#PWR?" H 8250 2270 30  0001 C CNN
+F 1 "+12P" H 8250 2400 30  0000 C CNN
+F 2 "" H 8250 2300 60  0000 C CNN
+F 3 "" H 8250 2300 60  0000 C CNN
+	1    8250 2300
 	1    0    0    -1
 $EndComp
@@
 L GND #PWR?
 U 1 1 52F684D0
-P 9050 2700
-F 0 "#PWR?" H 9050 2700 30  0001 C CNN
-F 1 "GND" H 9050 2630 30  0001 C CNN
-F 2 "" H 9050 2700 60  0000 C CNN
-F 3 "" H 9050 2700 60  0000 C CNN
-	1    9050 2700
+P 9150 3200
+F 0 "#PWR?" H 9150 3200 30  0001 C CNN
+F 1 "GND" H 9150 3130 30  0001 C CNN
+F 2 "" H 9150 3200 60  0000 C CNN
+F 3 "" H 9150 3200 60  0000 C CNN
+	1    9150 3200
 	1    0    0    -1
 $EndComp
@@
 L -12P #PWR?
 U 1 1 52F684D6
-P 8150 3700
-F 0 "#PWR?" H 8150 3830 20  0001 C CNN
-F 1 "-12P" H 8150 3800 30  0000 C CNN
-F 2 "" H 8150 3700 60  0000 C CNN
-F 3 "" H 8150 3700 60  0000 C CNN
-	1    8150 3700
+P 8250 4200
+F 0 "#PWR?" H 8250 4330 20  0001 C CNN
+F 1 "-12P" H 8250 4300 30  0000 C CNN
+F 2 "" H 8250 4200 60  0000 C CNN
+F 3 "" H 8250 4200 60  0000 C CNN
+	1    8250 4200
 	-1   0    0    1
 $EndComp
@@
 L INDUCTOR L?
 U 1 1 52F684DE
-P 8700 2050
-F 0 "L?" V 8650 2050 40  0000 C CNN
-F 1 "INDUCTOR" V 8800 2050 40  0000 C CNN
-F 2 "~" H 8700 2050 60  0000 C CNN
-F 3 "~" H 8700 2050 60  0000 C CNN
-	1    8700 2050
+P 8800 2550
+F 0 "L?" V 8750 2550 40  0000 C CNN
+F 1 "INDUCTOR" V 8900 2550 40  0000 C CNN
+F 2 "~" H 8800 2550 60  0000 C CNN
+F 3 "~" H 8800 2550 60  0000 C CNN
+	1    8800 2550
 	0    -1   -1   0
 $EndComp
@@
 L INDUCTOR L?
 U 1 1 52F684EB
-P 8800 3450
-F 0 "L?" V 8750 3450 40  0000 C CNN
-F 1 "INDUCTOR" V 8900 3450 40  0000 C CNN
-F 2 "~" H 8800 3450 60  0000 C CNN
-F 3 "~" H 8800 3450 60  0000 C CNN
-	1    8800 3450
+P 8900 3950
+F 0 "L?" V 8850 3950 40  0000 C CNN
+F 1 "INDUCTOR" V 9000 3950 40  0000 C CNN
+F 2 "~" H 8900 3950 60  0000 C CNN
+F 3 "~" H 8900 3950 60  0000 C CNN
+	1    8900 3950
 	0    1    1    0
 $EndComp
@@
 L C C?
 U 1 1 52F68508
-P 9450 2300
-F 0 "C?" H 9450 2400 40  0000 L CNN
-F 1 "C" H 9456 2215 40  0000 L CNN
-F 2 "~" H 9488 2150 30  0000 C CNN
-F 3 "~" H 9450 2300 60  0000 C CNN
-	1    9450 2300
+P 9550 2800
+F 0 "C?" H 9550 2900 40  0000 L CNN
+F 1 "C" H 9556 2715 40  0000 L CNN
+F 2 "~" H 9588 2650 30  0000 C CNN
+F 3 "~" H 9550 2800 60  0000 C CNN
+	1    9550 2800
 	1    0    0    -1
 $EndComp
@@
 L C C?
 U 1 1 52F68515
-P 9450 3000
-F 0 "C?" H 9450 3100 40  0000 L CNN
-F 1 "C" H 9456 2915 40  0000 L CNN
-F 2 "~" H 9488 2850 30  0000 C CNN
-F 3 "~" H 9450 3000 60  0000 C CNN
-	1    9450 3000
-	1    0    0    -1
-$EndComp
-Wire Wire Line
-	9050 2700 9050 2650
-Wire Wire Line
-	9050 2650 9450 2650
-Wire Wire Line
-	9450 2500 9450 2800
-Connection ~ 9450 2650
-Wire Wire Line
-	9100 3450 10000 3450
-Wire Wire Line
-	9450 3450 9450 3200
-Wire Wire Line
-	9050 2050 10100 2050
-Wire Wire Line
-	9450 2050 9450 2100
-Wire Wire Line
-	8150 1800 8150 2050
-Wire Wire Line
-	8150 2050 8400 2050
-Wire Wire Line
-	8150 3700 8150 3450
-Wire Wire Line
-	8150 3450 8500 3450
+P 9550 3500
+F 0 "C?" H 9550 3600 40  0000 L CNN
+F 1 "C" H 9556 3415 40  0000 L CNN
+F 2 "~" H 9588 3350 30  0000 C CNN
+F 3 "~" H 9550 3500 60  0000 C CNN
+	1    9550 3500
+	1    0    0    -1
+$EndComp
+Wire Wire Line
+	9150 3200 9150 3150
+Wire Wire Line
+	9150 3150 9550 3150
+Wire Wire Line
+	9550 3000 9550 3300
+Connection ~ 9550 3150
+Wire Wire Line
+	9200 3950 10100 3950
+Wire Wire Line
+	9550 3950 9550 3700
+Wire Wire Line
+	9100 2550 10200 2550
+Wire Wire Line
+	9550 2550 9550 2600
+Wire Wire Line
+	8250 2300 8250 2550
+Wire Wire Line
+	8250 2550 8500 2550
+Wire Wire Line
+	8250 4200 8250 3950
+Wire Wire Line
+	8250 3950 8600 3950
 $Comp
 L -12V #PWR?
 U 1 1 52F68656
-P 10000 3700
-F 0 "#PWR?" H 10000 3830 20  0001 C CNN
-F 1 "-12V" H 10000 3800 30  0000 C CNN
-F 2 "" H 10000 3700 60  0000 C CNN
-F 3 "" H 10000 3700 60  0000 C CNN
-	1    10000 3700
+P 10100 4200
+F 0 "#PWR?" H 10100 4330 20  0001 C CNN
+F 1 "-12V" H 10100 4300 30  0000 C CNN
+F 2 "" H 10100 4200 60  0000 C CNN
+F 3 "" H 10100 4200 60  0000 C CNN
+	1    10100 4200
 	-1   0    0    1
 $EndComp
@@
 L +12V #PWR?
 U 1 1 52F68665
-P 10100 1750
-F 0 "#PWR?" H 10100 1700 20  0001 C CNN
-F 1 "+12V" H 10100 1850 30  0000 C CNN
-F 2 "" H 10100 1750 60  0000 C CNN
-F 3 "" H 10100 1750 60  0000 C CNN
-	1    10100 1750
-	1    0    0    -1
-$EndComp
-Wire Wire Line
-	10100 2050 10100 1750
-Connection ~ 9450 2050
-Wire Wire Line
-	10000 3450 10000 3700
-Connection ~ 9450 3450
+P 10200 2250
+F 0 "#PWR?" H 10200 2200 20  0001 C CNN
+F 1 "+12V" H 10200 2350 30  0000 C CNN
+F 2 "" H 10200 2250 60  0000 C CNN
+F 3 "" H 10200 2250 60  0000 C CNN
+	1    10200 2250
+	1    0    0    -1
+$EndComp
+Wire Wire Line
+	10200 2550 10200 2250
+Connection ~ 9550 2550
+Wire Wire Line
+	10100 3950 10100 4200
+Connection ~ 9550 3950
 $Comp
 L +12C #PWR?
@@
 	0    -1   -1   0
 $EndComp
+$Comp
+L +5P #PWR?
+U 1 1 5302A929
+P 5000 1550
+F 0 "#PWR?" H 5000 1680 20  0001 C CNN
+F 1 "+5P" H 5000 1650 30  0000 C CNN
+F 2 "" H 5000 1550 60  0000 C CNN
+F 3 "" H 5000 1550 60  0000 C CNN
+	1    5000 1550
+	1    0    0    -1
+$EndComp
+$Comp
+L +3.3VP #PWR?
+U 1 1 5302A942
+P 4300 1550
+F 0 "#PWR?" H 4350 1580 20  0001 C CNN
+F 1 "+3.3VP" H 4300 1640 30  0000 C CNN
+F 2 "" H 4300 1550 60  0000 C CNN
+F 3 "" H 4300 1550 60  0000 C CNN
+	1    4300 1550
+	1    0    0    -1
+$EndComp
+$Comp
+L INDUCTOR L?
+U 1 1 5302A984
+P 8700 1000
+F 0 "L?" V 8650 1000 40  0000 C CNN
+F 1 "INDUCTOR" V 8800 1000 40  0000 C CNN
+F 2 "~" H 8700 1000 60  0000 C CNN
+F 3 "~" H 8700 1000 60  0000 C CNN
+	1    8700 1000
+	0    -1   -1   0
+$EndComp
+$Comp
+L C C?
+U 1 1 5302A98A
+P 9450 1250
+F 0 "C?" H 9450 1350 40  0000 L CNN
+F 1 "C" H 9456 1165 40  0000 L CNN
+F 2 "~" H 9488 1100 30  0000 C CNN
+F 3 "~" H 9450 1250 60  0000 C CNN
+	1    9450 1250
+	1    0    0    -1
+$EndComp
+Wire Wire Line
+	9000 1000 10100 1000
+Wire Wire Line
+	9450 1000 9450 1050
+Wire Wire Line
+	8150 750  8150 1000
+Wire Wire Line
+	8150 1000 8400 1000
+Wire Wire Line
+	10100 1000 10100 700
+Connection ~ 9450 1000
+$Comp
+L GND #PWR?
+U 1 1 5302A99D
+P 9450 1600
+F 0 "#PWR?" H 9450 1600 30  0001 C CNN
+F 1 "GND" H 9450 1530 30  0001 C CNN
+F 2 "" H 9450 1600 60  0000 C CNN
+F 3 "" H 9450 1600 60  0000 C CNN
+	1    9450 1600
+	1    0    0    -1
+$EndComp
+Wire Wire Line
+	9450 1600 9450 1450
+$Comp
+L +5P #PWR?
+U 1 1 5302A9DA
+P 8150 750
+F 0 "#PWR?" H 8150 880 20  0001 C CNN
+F 1 "+5P" H 8150 850 30  0000 C CNN
+F 2 "" H 8150 750 60  0000 C CNN
+F 3 "" H 8150 750 60  0000 C CNN
+	1    8150 750
+	1    0    0    -1
+$EndComp
+$Comp
+L +5V #PWR?
+U 1 1 5302A9E9
+P 10100 700
+F 0 "#PWR?" H 10100 790 20  0001 C CNN
+F 1 "+5V" H 10100 790 30  0000 C CNN
+F 2 "" H 10100 700 60  0000 C CNN
+F 3 "" H 10100 700 60  0000 C CNN
+	1    10100 700
+	1    0    0    -1
+$EndComp
 $EndSCHEMATC
