File: Relay.sch (KiCad schematic (older format))
At the start: 0 parts

Commit message: Created CurrentDriver, Relay, and PowerProtection modules
Parts:
- added D?: LED, ~, symbol LED
- added D?: DIODE, ~, symbol DIODE
- added K?: SPDT_RELAY, ~, symbol SPDT_RELAY
- added Q?: NPN, ~, symbol NPN
- added R? (x5): R, ~, symbol R
- added U?: PHTRANS, ~, symbol PHTRANS
Connections:
- net labels added: +12P, COM, GND, NC, NO
- net labels removed: Relay+, Relay-
- wire segments 0 -> 26
Changed lines of the file:
@@
 LIBS:contrib
 LIBS:valves
+LIBS:BenchBudEE
 LIBS:BenchBudEE-cache
 EELAYER 27 0
@@
 $Descr A4 11693 8268
 encoding utf-8
-Sheet 4 8
+Sheet 4 9
 Title ""
-Date "6 feb 2014"
+Date "9 feb 2014"
 Rev ""
 Comp ""
@@
 Comment4 ""
 $EndDescr
-Text HLabel 3350 2500 0    60   Input ~ 0
+Text HLabel 4150 3450 0    60   Input ~ 0
 DIN+
-Text HLabel 3350 3200 0    60   Output ~ 0
+Text HLabel 4150 3800 0    60   Output ~ 0
 DIN-
-Text HLabel 8500 2400 0    60   Input ~ 0
-Relay+
-Text HLabel 8500 2950 0    60   Output ~ 0
-Relay-
+Text HLabel 10250 2700 2    60   BiDi ~ 0
+NC
+Text HLabel 10250 2900 2    60   BiDi ~ 0
+NO
+$Comp
+L PHTRANS U?
+U 1 1 52F67364
+P 5850 3650
+F 0 "U?" H 5800 4000 70  0000 C CNN
+F 1 "PHTRANS" H 5800 3300 70  0000 C CNN
+F 2 "~" H 5850 3650 60  0000 C CNN
+F 3 "~" H 5850 3650 60  0000 C CNN
+	1    5850 3650
+	1    0    0    -1
+$EndComp
+$Comp
+L R R?
+U 1 1 52F67373
+P 7000 3850
+F 0 "R?" V 7080 3850 40  0000 C CNN
+F 1 "R" V 7007 3851 40  0000 C CNN
+F 2 "~" V 6930 3850 30  0000 C CNN
+F 3 "~" H 7000 3850 30  0000 C CNN
+	1    7000 3850
+	0    -1   -1   0
+$EndComp
+$Comp
+L NPN Q?
+U 1 1 52F67382
+P 8800 3850
+F 0 "Q?" H 8800 3700 50  0000 R CNN
+F 1 "NPN" H 8800 4000 50  0000 R CNN
+F 2 "~" H 8800 3850 60  0000 C CNN
+F 3 "~" H 8800 3850 60  0000 C CNN
+	1    8800 3850
+	1    0    0    -1
+$EndComp
+$Comp
+L LED D?
+U 1 1 52F6739B
+P 6600 4300
+F 0 "D?" H 6600 4400 50  0000 C CNN
+F 1 "LED" H 6600 4200 50  0000 C CNN
+F 2 "~" H 6600 4300 60  0000 C CNN
+F 3 "~" H 6600 4300 60  0000 C CNN
+	1    6600 4300
+	0    1    1    0
+$EndComp
+$Comp
+L SPDT_RELAY K?
+U 1 1 52F67845
+P 9650 2750
+F 0 "K?" H 9650 3050 70  0000 C CNN
+F 1 "SPDT_RELAY" H 9650 2100 70  0000 C CNN
+F 2 "~" H 9650 2750 60  0000 C CNN
+F 3 "~" H 9650 2750 60  0000 C CNN
+	1    9650 2750
+	1    0    0    -1
+$EndComp
+Text HLabel 10250 2050 2    60   BiDi ~ 0
+COM
+$Comp
+L R R?
+U 1 1 52F678EA
+P 8900 4650
+F 0 "R?" V 8980 4650 40  0000 C CNN
+F 1 "R" V 8907 4651 40  0000 C CNN
+F 2 "~" V 8830 4650 30  0000 C CNN
+F 3 "~" H 8900 4650 30  0000 C CNN
+	1    8900 4650
+	1    0    0    -1
+$EndComp
+$Comp
+L GND #PWR?
+U 1 1 52F678FD
+P 8900 5250
+F 0 "#PWR?" H 8900 5250 30  0001 C CNN
+F 1 "GND" H 8900 5180 30  0001 C CNN
+F 2 "" H 8900 5250 60  0000 C CNN
+F 3 "" H 8900 5250 60  0000 C CNN
+	1    8900 5250
+	1    0    0    -1
+$EndComp
+$Comp
+L R R?
+U 1 1 52F67935
+P 6600 4850
+F 0 "R?" V 6680 4850 40  0000 C CNN
+F 1 "R" V 6607 4851 40  0000 C CNN
+F 2 "~" V 6530 4850 30  0000 C CNN
+F 3 "~" H 6600 4850 30  0000 C CNN
+	1    6600 4850
+	1    0    0    -1
+$EndComp
+$Comp
+L R R?
+U 1 1 52F6798E
+P 6750 3450
+F 0 "R?" V 6830 3450 40  0000 C CNN
+F 1 "R" V 6757 3451 40  0000 C CNN
+F 2 "~" V 6680 3450 30  0000 C CNN
+F 3 "~" H 6750 3450 30  0000 C CNN
+	1    6750 3450
+	0    -1   -1   0
+$EndComp
+$Comp
+L R R?
+U 1 1 52F679BD
+P 4700 3800
+F 0 "R?" V 4780 3800 40  0000 C CNN
+F 1 "R" V 4707 3801 40  0000 C CNN
+F 2 "~" V 4630 3800 30  0000 C CNN
+F 3 "~" H 4700 3800 30  0000 C CNN
+	1    4700 3800
+	0    -1   -1   0
+$EndComp
+$Comp
+L DIODE D?
+U 1 1 52F67A2F
+P 8100 3300
+F 0 "D?" H 8100 3400 40  0000 C CNN
+F 1 "DIODE" H 8100 3200 40  0000 C CNN
+F 2 "~" H 8100 3300 60  0000 C CNN
+F 3 "~" H 8100 3300 60  0000 C CNN
+	1    8100 3300
+	0    -1   -1   0
+$EndComp
+Wire Wire Line
+	10250 2900 10050 2900
+Wire Wire Line
+	10250 2700 10050 2700
+Wire Wire Line
+	6400 3850 6750 3850
+Wire Wire Line
+	7250 3850 8600 3850
+Wire Wire Line
+	8900 4050 8900 4400
+Wire Wire Line
+	9250 3100 8900 3100
+Wire Wire Line
+	8900 3100 8900 3650
+Wire Wire Line
+	7100 3000 9250 3000
+Wire Wire Line
+	7100 2500 7100 3650
+Wire Wire Line
+	8900 4900 8900 5250
+Wire Wire Line
+	6600 4100 6600 3850
+Connection ~ 6600 3850
+Wire Wire Line
+	6600 4600 6600 4500
+Wire Wire Line
+	6600 5100 6600 5150
+Wire Wire Line
+	6600 5150 8900 5150
+Connection ~ 8900 5150
+Wire Wire Line
+	7100 3650 6400 3650
+Connection ~ 7100 3000
+Wire Wire Line
+	6500 3450 6400 3450
+Wire Wire Line
+	7000 3450 7100 3450
+Connection ~ 7100 3450
+Wire Wire Line
+	4950 3800 5300 3800
+Wire Wire Line
+	4150 3450 5300 3450
+Wire Wire Line
+	4150 3800 4450 3800
+Wire Wire Line
+	10250 2050 9050 2050
+Wire Wire Line
+	9050 2050 9050 2800
+Wire Wire Line
+	9050 2800 9250 2800
+Wire Wire Line
+	8100 3100 8100 3000
+Connection ~ 8100 3000
+Wire Wire Line
+	8100 3500 8100 3600
+Wire Wire Line
+	8100 3600 8900 3600
+Connection ~ 8900 3600
+$Comp
+L +12P #PWR?
+U 1 1 52F68137
+P 7100 2500
+F 0 "#PWR?" H 7100 2470 30  0001 C CNN
+F 1 "+12P" H 7100 2600 30  0000 C CNN
+F 2 "" H 7100 2500 60  0000 C CNN
+F 3 "" H 7100 2500 60  0000 C CNN
+	1    7100 2500
+	1    0    0    -1
+$EndComp
 $EndSCHEMATC

Commit message: Current driver refactoring, LED module, Arduino
Connections:
- net labels added: RELAY+, RELAY-, RELAY_COM, RELAY_NC, RELAY_NO
- net labels removed: COM, DIN+, DIN-, NC, NO
Changed lines of the file:
@@
 $Descr A4 11693 8268
 encoding utf-8
-Sheet 4 9
+Sheet 3 9
 Title ""
 Date "9 feb 2014"
@@
 $EndDescr
 Text HLabel 4150 3450 0    60   Input ~ 0
-DIN+
+RELAY+
 Text HLabel 4150 3800 0    60   Output ~ 0
-DIN-
+RELAY-
 Text HLabel 10250 2700 2    60   BiDi ~ 0
-NC
+RELAY_NC
 Text HLabel 10250 2900 2    60   BiDi ~ 0
-NO
+RELAY_NO
 $Comp
 L PHTRANS U?
@@
 $EndComp
 Text HLabel 10250 2050 2    60   BiDi ~ 0
-COM
+RELAY_COM
 $Comp
 L R R?

Commit message: Relay module association and placement
Parts:
- removed R?: R, ~, symbol R
- removed U?: PHTRANS, ~, symbol PHTRANS
- added R3, R5: 0, ~, symbol R
- added U1: LTV-816S, symbol OPTO-TRANSISTOR4
- D1: renamed from D?; value LED -> LG Q971-KN-1
- D2: renamed from D?; value DIODE -> B130; MFG Part Number (none) -> B130-13-F
- K1: renamed from K?; value SPDT_RELAY -> 1461069-5
- Q1: renamed from Q?; value NPN -> 2N3904; MFG Name (none) -> Diodes Inc; MFG Part Number (none) -> MMBT3904-7-F
- R1: renamed from R?; value R -> 500
- R2: renamed from R?; value R -> 200
- R4: renamed from R?; value R -> 100
- R6: renamed from R?; value R -> 0
Connections:
- wire segments 26 -> 27
Other:
- moved on the sheet: R1, R4
Changed lines of the file:
@@
 $Descr A4 11693 8268
 encoding utf-8
-Sheet 3 9
+Sheet 9 9
 Title ""
-Date "18 feb 2014"
+Date "20 feb 2014"
 Rev ""
 Comp ""
@@
 Comment4 ""
 $EndDescr
-Text HLabel 4150 3450 0    60   Input ~ 0
+Text HLabel 3850 3550 0    60   Input ~ 0
 RELAY+
-Text HLabel 4150 3800 0    60   Output ~ 0
+Text HLabel 3850 3850 0    60   Output ~ 0
 RELAY-
 Text HLabel 10250 2700 2    60   BiDi ~ 0
@@
 RELAY_NO
 $Comp
-L PHTRANS U?
-U 1 1 52F67364
-P 5850 3650
-F 0 "U?" H 5800 4000 70  0000 C CNN
-F 1 "PHTRANS" H 5800 3300 70  0000 C CNN
-F 2 "~" H 5850 3650 60  0000 C CNN
-F 3 "~" H 5850 3650 60  0000 C CNN
-	1    5850 3650
-	1    0    0    -1
-$EndComp
-$Comp
-L R R?
+L R R4
 U 1 1 52F67373
-P 7000 3850
-F 0 "R?" V 7080 3850 40  0000 C CNN
-F 1 "R" V 7007 3851 40  0000 C CNN
-F 2 "~" V 6930 3850 30  0000 C CNN
-F 3 "~" H 7000 3850 30  0000 C CNN
-	1    7000 3850
+P 7400 3850
+F 0 "R4" V 7480 3850 40  0000 C CNN
+F 1 "100" V 7407 3851 40  0000 C CNN
+F 2 "~" V 7330 3850 30  0000 C CNN
+F 3 "~" H 7400 3850 30  0000 C CNN
+	1    7400 3850
 	0    -1   -1   0
 $EndComp
 $Comp
-L NPN Q?
+L NPN Q1
 U 1 1 52F67382
 P 8800 3850
-F 0 "Q?" H 8800 3700 50  0000 R CNN
-F 1 "NPN" H 8800 4000 50  0000 R CNN
+F 0 "Q1" H 8800 3700 50  0000 R CNN
+F 1 "2N3904" H 8800 4000 50  0000 R CNN
 F 2 "~" H 8800 3850 60  0000 C CNN
 F 3 "~" H 8800 3850 60  0000 C CNN
+F 4 "Diodes Inc" H 8800 3850 60  0001 C CNN "MFG Name"
+F 5 "MMBT3904-7-F" H 8800 3850 60  0001 C CNN "MFG Part Number"
 	1    8800 3850
 	1    0    0    -1
 $EndComp
 $Comp
-L LED D?
+L LED D1
 U 1 1 52F6739B
 P 6600 4300
-F 0 "D?" H 6600 4400 50  0000 C CNN
-F 1 "LED" H 6600 4200 50  0000 C CNN
+F 0 "D1" H 6600 4400 50  0000 C CNN
+F 1 "LG Q971-KN-1" H 6600 4200 50  0000 C CNN
 F 2 "~" H 6600 4300 60  0000 C CNN
 F 3 "~" H 6600 4300 60  0000 C CNN
@@
 $EndComp
 $Comp
-L SPDT_RELAY K?
+L SPDT_RELAY K1
 U 1 1 52F67845
 P 9650 2750
-F 0 "K?" H 9650 3050 70  0000 C CNN
-F 1 "SPDT_RELAY" H 9650 2100 70  0000 C CNN
+F 0 "K1" H 9650 3050 70  0000 C CNN
+F 1 "1461069-5" H 9650 2100 70  0000 C CNN
 F 2 "~" H 9650 2750 60  0000 C CNN
 F 3 "~" H 9650 2750 60  0000 C CNN
@@
 RELAY_COM
 $Comp
-L R R?
+L R R6
 U 1 1 52F678EA
 P 8900 4650
-F 0 "R?" V 8980 4650 40  0000 C CNN
-F 1 "R" V 8907 4651 40  0000 C CNN
+F 0 "R6" V 8980 4650 40  0000 C CNN
+F 1 "0" V 8907 4651 40  0000 C CNN
 F 2 "~" V 8830 4650 30  0000 C CNN
 F 3 "~" H 8900 4650 30  0000 C CNN
@@
 $EndComp
 $Comp
-L GND #PWR?
+L GND #PWR051
 U 1 1 52F678FD
 P 8900 5250
-F 0 "#PWR?" H 8900 5250 30  0001 C CNN
+F 0 "#PWR051" H 8900 5250 30  0001 C CNN
 F 1 "GND" H 8900 5180 30  0001 C CNN
 F 2 "" H 8900 5250 60  0000 C CNN
@@
 $EndComp
 $Comp
-L R R?
+L R R2
 U 1 1 52F67935
 P 6600 4850
-F 0 "R?" V 6680 4850 40  0000 C CNN
-F 1 "R" V 6607 4851 40  0000 C CNN
+F 0 "R2" V 6680 4850 40  0000 C CNN
+F 1 "200" V 6607 4851 40  0000 C CNN
 F 2 "~" V 6530 4850 30  0000 C CNN
 F 3 "~" H 6600 4850 30  0000 C CNN
@@
 $EndComp
 $Comp
-L R R?
-U 1 1 52F6798E
-P 6750 3450
-F 0 "R?" V 6830 3450 40  0000 C CNN
-F 1 "R" V 6757 3451 40  0000 C CNN
-F 2 "~" V 6680 3450 30  0000 C CNN
-F 3 "~" H 6750 3450 30  0000 C CNN
-	1    6750 3450
+L R R1
+U 1 1 52F679BD
+P 4400 3850
+F 0 "R1" V 4480 3850 40  0000 C CNN
+F 1 "500" V 4407 3851 40  0000 C CNN
+F 2 "~" V 4330 3850 30  0000 C CNN
+F 3 "~" H 4400 3850 30  0000 C CNN
+	1    4400 3850
 	0    -1   -1   0
 $EndComp
 $Comp
-L R R?
-U 1 1 52F679BD
-P 4700 3800
-F 0 "R?" V 4780 3800 40  0000 C CNN
-F 1 "R" V 4707 3801 40  0000 C CNN
-F 2 "~" V 4630 3800 30  0000 C CNN
-F 3 "~" H 4700 3800 30  0000 C CNN
-	1    4700 3800
-	0    -1   -1   0
-$EndComp
-$Comp
-L DIODE D?
+L DIODE D2
 U 1 1 52F67A2F
 P 8100 3300
-F 0 "D?" H 8100 3400 40  0000 C CNN
-F 1 "DIODE" H 8100 3200 40  0000 C CNN
+F 0 "D2" H 8100 3400 40  0000 C CNN
+F 1 "B130" H 8100 3200 40  0000 C CNN
 F 2 "~" H 8100 3300 60  0000 C CNN
 F 3 "~" H 8100 3300 60  0000 C CNN
+F 4 "B130-13-F" H 8100 3300 60  0001 C CNN "MFG Part Number"
 	1    8100 3300
 	0    -1   -1   0
@@
 	10250 2700 10050 2700
 Wire Wire Line
-	6400 3850 6750 3850
-Wire Wire Line
-	7250 3850 8600 3850
+	6400 3850 7150 3850
+Wire Wire Line
+	7650 3850 8600 3850
 Wire Wire Line
 	8900 4050 8900 4400
@@
 	8900 3100 8900 3650
 Wire Wire Line
-	7100 3000 9250 3000
-Wire Wire Line
-	7100 2500 7100 3650
+	8100 3000 9250 3000
 Wire Wire Line
 	8900 4900 8900 5250
@@
 Connection ~ 8900 5150
 Wire Wire Line
-	7100 3650 6400 3650
-Connection ~ 7100 3000
-Wire Wire Line
-	6500 3450 6400 3450
-Wire Wire Line
-	7000 3450 7100 3450
-Connection ~ 7100 3450
-Wire Wire Line
-	4950 3800 5300 3800
-Wire Wire Line
-	4150 3450 5300 3450
-Wire Wire Line
-	4150 3800 4450 3800
+	7100 3550 6400 3550
+Wire Wire Line
+	4650 3850 5150 3850
+Wire Wire Line
+	3850 3550 5150 3550
+Wire Wire Line
+	3850 3850 4150 3850
 Wire Wire Line
 	10250 2050 9050 2050
@@
 	9050 2800 9250 2800
 Wire Wire Line
-	8100 3100 8100 3000
+	8100 2900 8100 3100
 Connection ~ 8100 3000
 Wire Wire Line
@@
 Connection ~ 8900 3600
 $Comp
-L +12P #PWR?
+L +12P #PWR052
 U 1 1 52F68137
-P 7100 2500
-F 0 "#PWR?" H 7100 2470 30  0001 C CNN
-F 1 "+12P" H 7100 2600 30  0000 C CNN
-F 2 "" H 7100 2500 60  0000 C CNN
-F 3 "" H 7100 2500 60  0000 C CNN
-	1    7100 2500
-	1    0    0    -1
-$EndComp
+P 7100 2250
+F 0 "#PWR052" H 7100 2220 30  0001 C CNN
+F 1 "+12P" H 7100 2350 30  0000 C CNN
+F 2 "" H 7100 2250 60  0000 C CNN
+F 3 "" H 7100 2250 60  0000 C CNN
+	1    7100 2250
+	1    0    0    -1
+$EndComp
+$Comp
+L OPTO-TRANSISTOR4 U1
+U 1 1 53056D08
+P 5800 3700
+F 0 "U1" H 6000 3950 60  0000 C CNN
+F 1 "LTV-816S" H 5800 3450 60  0000 C CNN
+F 2 "" H 5800 3700 60  0000 C CNN
+F 3 "" H 5800 3700 60  0000 C CNN
+F 4 "LTV-816S" H 5800 3700 60  0001 C CNN "MFG Part Number"
+	1    5800 3700
+	1    0    0    -1
+$EndComp
+$Comp
+L R R3
+U 1 1 53056E42
+P 7100 2650
+F 0 "R3" V 7180 2650 40  0000 C CNN
+F 1 "0" V 7107 2651 40  0000 C CNN
+F 2 "~" V 7030 2650 30  0000 C CNN
+F 3 "~" H 7100 2650 30  0000 C CNN
+	1    7100 2650
+	-1   0    0    1
+$EndComp
+Wire Wire Line
+	7100 2250 7100 2400
+Wire Wire Line
+	7100 2900 7100 3550
+$Comp
+L R R5
+U 1 1 53056E84
+P 8100 2650
+F 0 "R5" V 8180 2650 40  0000 C CNN
+F 1 "0" V 8107 2651 40  0000 C CNN
+F 2 "~" V 8030 2650 30  0000 C CNN
+F 3 "~" H 8100 2650 30  0000 C CNN
+	1    8100 2650
+	-1   0    0    1
+$EndComp
+Wire Wire Line
+	8100 2400 8100 2350
+Wire Wire Line
+	8100 2350 7100 2350
+Connection ~ 7100 2350
 $EndSCHEMATC

Commit message: Fan driver: assc/placement
Parts:
- D2: value B130 -> B130-13-F; MFG Name (none) -> Diodes Inc
Changed lines of the file:
@@
 $Descr A4 11693 8268
 encoding utf-8
-Sheet 9 9
+Sheet 7 9
 Title ""
-Date "22 feb 2014"
+Date "23 feb 2014"
 Rev ""
 Comp ""
@@
 $EndComp
 $Comp
-L GND #PWR45
+L GND #PWR041
 U 1 1 52F678FD
 P 8900 5250
-F 0 "#PWR45" H 8900 5250 30  0001 C CNN
+F 0 "#PWR041" H 8900 5250 30  0001 C CNN
 F 1 "GND" H 8900 5180 30  0001 C CNN
 F 2 "" H 8900 5250 60  0000 C CNN
@@
 P 8100 3300
 F 0 "D2" H 8100 3400 40  0000 C CNN
-F 1 "B130" H 8100 3200 40  0000 C CNN
+F 1 "B130-13-F" H 8100 3200 40  0000 C CNN
 F 2 "~" H 8100 3300 60  0000 C CNN
 F 3 "~" H 8100 3300 60  0000 C CNN
-F 4 "B130-13-F" H 8100 3300 60  0001 C CNN "MFG Part Number"
+F 4 "Diodes Inc" H 8100 3300 60  0001 C CNN "MFG Name"
+F 5 "B130-13-F" H 8100 3300 60  0001 C CNN "MFG Part Number"
 	1    8100 3300
 	0    -1   -1   0
@@
 Connection ~ 8900 3600
 $Comp
-L +12P #PWR44
+L +12P #PWR042
 U 1 1 52F68137
 P 7100 2250
-F 0 "#PWR44" H 7100 2220 30  0001 C CNN
+F 0 "#PWR042" H 7100 2220 30  0001 C CNN
 F 1 "+12P" H 7100 2350 30  0000 C CNN
 F 2 "" H 7100 2250 60  0000 C CNN
