File: Thermocouple.sch (KiCad schematic (older format))
At the start: 15 parts

Commit message: Refactoring and Created key shortcuts
Changed lines of the file:
@@
 $Descr A4 11693 8268
 encoding utf-8
-Sheet 3 9
+Sheet 2 9
 Title ""
-Date "9 feb 2014"
+Date "18 feb 2014"
 Rev ""
 Comp ""
@@
 Wire Wire Line
 	10400 5750 10400 6100
-$Comp
-L -12V #PWR?
-U 1 1 52F32F37
-P 10400 6550
-F 0 "#PWR?" H 10400 6680 20  0001 C CNN
-F 1 "-12V" H 10400 6650 30  0000 C CNN
-F 2 "" H 10400 6550 60  0000 C CNN
-F 3 "" H 10400 6550 60  0000 C CNN
-	1    10400 6550
-	-1   0    0    1
-$EndComp
-Wire Wire Line
-	10400 6550 10400 6500
+Wire Wire Line
+	10400 6500 10400 6600
 Wire Wire Line
 	8950 6050 10400 6050
@@
 Text Notes 2350 2900 0    60   ~ 0
 16-24 Bit ADC
+$Comp
+L AGND #PWR?
+U 1 1 5302CE9A
+P 10400 6600
+F 0 "#PWR?" H 10400 6600 40  0001 C CNN
+F 1 "AGND" H 10400 6530 50  0000 C CNN
+F 2 "" H 10400 6600 60  0000 C CNN
+F 3 "" H 10400 6600 60  0000 C CNN
+	1    10400 6600
+	1    0    0    -1
+$EndComp
 $EndSCHEMATC

Commit message: Relay module association and placement
Parts:
- gave numbers to parts that had none: 12
Changed lines of the file:
@@
 Sheet 2 9
 Title ""
-Date "18 feb 2014"
+Date "20 feb 2014"
 Rev ""
 Comp ""
@@
 CS_N
 $Comp
-L LM324 U?
-U 1 1 52F32905
+L LM324 U4
+U 3 1 52F32905
 P 9450 2300
-F 0 "U?" H 9500 2500 60  0000 C CNN
+F 0 "U4" H 9500 2500 60  0000 C CNN
 F 1 "LM324" H 9600 2100 50  0000 C CNN
 F 2 "" H 9450 2300 60  0000 C CNN
 F 3 "" H 9450 2300 60  0000 C CNN
-	1    9450 2300
+	3    9450 2300
 	-1   0    0    -1
 $EndComp
 $Comp
-L LM324 U?
-U 1 1 52F3292B
+L LM324 U4
+U 4 1 52F3292B
 P 9450 4700
-F 0 "U?" H 9500 4900 60  0000 C CNN
+F 0 "U4" H 9500 4900 60  0000 C CNN
 F 1 "LM324" H 9600 4500 50  0000 C CNN
 F 2 "" H 9450 4700 60  0000 C CNN
 F 3 "" H 9450 4700 60  0000 C CNN
-	1    9450 4700
+	4    9450 4700
 	-1   0    0    1
 $EndComp
 $Comp
-L LM324 U?
+L LM324 U4
 U 1 1 52F32931
 P 7250 3550
-F 0 "U?" H 7300 3750 60  0000 C CNN
+F 0 "U4" H 7300 3750 60  0000 C CNN
 F 1 "LM324" H 7400 3350 50  0000 C CNN
 F 2 "" H 7250 3550 60  0000 C CNN
@@
 $EndComp
 $Comp
-L LM324 U?
-U 1 1 52F32937
+L LM324 U4
+U 2 1 52F32937
 P 8450 6150
-F 0 "U?" H 8500 6350 60  0000 C CNN
+F 0 "U4" H 8500 6350 60  0000 C CNN
 F 1 "LM324" H 8600 5950 50  0000 C CNN
 F 2 "" H 8450 6150 60  0000 C CNN
 F 3 "" H 8450 6150 60  0000 C CNN
-	1    8450 6150
+	2    8450 6150
 	-1   0    0    -1
 $EndComp
 $Comp
-L C C?
+L C C1
 U 1 1 52F3298A
 P 5050 6350
-F 0 "C?" H 5050 6450 40  0000 L CNN
+F 0 "C1" H 5050 6450 40  0000 L CNN
 F 1 "C" H 5056 6265 40  0000 L CNN
 F 2 "~" H 5088 6200 30  0000 C CNN
@@
 $EndComp
 $Comp
-L R R?
+L R R11
 U 1 1 52F32999
 P 8650 2850
-F 0 "R?" V 8730 2850 40  0000 C CNN
+F 0 "R11" V 8730 2850 40  0000 C CNN
 F 1 "R" V 8657 2851 40  0000 C CNN
 F 2 "~" V 8580 2850 30  0000 C CNN
@@
 $EndComp
 $Comp
-L R R?
+L R R12
 U 1 1 52F329A6
 P 8650 3500
-F 0 "R?" V 8730 3500 40  0000 C CNN
+F 0 "R12" V 8730 3500 40  0000 C CNN
 F 1 "R" V 8657 3501 40  0000 C CNN
 F 2 "~" V 8580 3500 30  0000 C CNN
@@
 $EndComp
 $Comp
-L R R?
+L R R13
 U 1 1 52F329AC
 P 8650 4200
-F 0 "R?" V 8730 4200 40  0000 C CNN
+F 0 "R13" V 8730 4200 40  0000 C CNN
 F 1 "R" V 8657 4201 40  0000 C CNN
 F 2 "~" V 8580 4200 30  0000 C CNN
@@
 	8350 4700 8950 4700
 $Comp
-L R R?
+L R R9
 U 1 1 52F329D3
 P 8100 2300
-F 0 "R?" V 8180 2300 40  0000 C CNN
+F 0 "R9" V 8180 2300 40  0000 C CNN
 F 1 "R" V 8107 2301 40  0000 C CNN
 F 2 "~" V 8030 2300 30  0000 C CNN
@@
 $EndComp
 $Comp
-L R R?
+L R R7
 U 1 1 52F329D9
 P 6400 2300
-F 0 "R?" V 6480 2300 40  0000 C CNN
+F 0 "R7" V 6480 2300 40  0000 C CNN
 F 1 "R" V 6407 2301 40  0000 C CNN
 F 2 "~" V 6330 2300 30  0000 C CNN
@@
 $EndComp
 $Comp
-L R R?
+L R R8
 U 1 1 52F329DF
 P 6400 4700
-F 0 "R?" V 6480 4700 40  0000 C CNN
+F 0 "R8" V 6480 4700 40  0000 C CNN
 F 1 "R" V 6407 4701 40  0000 C CNN
 F 2 "~" V 6330 4700 30  0000 C CNN
@@
 $EndComp
 $Comp
-L R R?
+L R R10
 U 1 1 52F329EF
 P 8100 4700
-F 0 "R?" V 8180 4700 40  0000 C CNN
+F 0 "R10" V 8180 4700 40  0000 C CNN
 F 1 "R" V 8107 4701 40  0000 C CNN
 F 2 "~" V 8030 4700 30  0000 C CNN
@@
 	10450 4800 9950 4800
 $Comp
-L +12V #PWR?
+L +12V #PWR01
 U 1 1 52F32ADE
 P 9550 1800
-F 0 "#PWR?" H 9550 1750 20  0001 C CNN
+F 0 "#PWR01" H 9550 1750 20  0001 C CNN
 F 1 "+12V" H 9550 1900 30  0000 C CNN
 F 2 "" H 9550 1800 60  0000 C CNN
@@
 	9550 1900 9550 1800
 $Comp
-L +12V #PWR?
+L +12V #PWR02
 U 1 1 52F32B09
 P 7350 4100
-F 0 "#PWR?" H 7350 4050 20  0001 C CNN
+F 0 "#PWR02" H 7350 4050 20  0001 C CNN
 F 1 "+12V" H 7350 4200 30  0000 C CNN
 F 2 "" H 7350 4100 60  0000 C CNN
@@
 $EndComp
 $Comp
-L +12V #PWR?
+L +12V #PWR03
 U 1 1 52F32B2F
 P 9550 5250
-F 0 "#PWR?" H 9550 5200 20  0001 C CNN
+F 0 "#PWR03" H 9550 5200 20  0001 C CNN
 F 1 "+12V" H 9550 5350 30  0000 C CNN
 F 2 "" H 9550 5250 60  0000 C CNN
@@
 $EndComp
 $Comp
-L -12V #PWR?
+L -12V #PWR04
 U 1 1 52F32B5A
 P 9550 2800
-F 0 "#PWR?" H 9550 2930 20  0001 C CNN
+F 0 "#PWR04" H 9550 2930 20  0001 C CNN
 F 1 "-12V" H 9550 2900 30  0000 C CNN
 F 2 "" H 9550 2800 60  0000 C CNN
@@
 $EndComp
 $Comp
-L -12V #PWR?
+L -12V #PWR05
 U 1 1 52F32B8D
 P 7350 3050
-F 0 "#PWR?" H 7350 3180 20  0001 C CNN
+F 0 "#PWR05" H 7350 3180 20  0001 C CNN
 F 1 "-12V" H 7350 3150 30  0000 C CNN
 F 2 "" H 7350 3050 60  0000 C CNN
@@
 	7350 3050 7350 3150
 $Comp
-L -12V #PWR?
+L -12V #PWR06
 U 1 1 52F32BE4
 P 9550 4200
-F 0 "#PWR?" H 9550 4330 20  0001 C CNN
+F 0 "#PWR06" H 9550 4330 20  0001 C CNN
 F 1 "-12V" H 9550 4300 30  0000 C CNN
 F 2 "" H 9550 4200 60  0000 C CNN
@@
 	9550 5250 9550 5100
 $Comp
-L AGND #PWR?
+L AGND #PWR07
 U 1 1 52F32CA2
 P 5950 5000
-F 0 "#PWR?" H 5950 5000 40  0001 C CNN
+F 0 "#PWR07" H 5950 5000 40  0001 C CNN
 F 1 "AGND" H 5950 4930 50  0000 C CNN
 F 2 "" H 5950 5000 60  0000 C CNN
@@
 	5950 4700 6150 4700
 $Comp
-L MCP3550-60-E/SN U?
+L MCP3550-60-E/SN U2
 U 1 1 52F32CDF
 P 2700 3700
-F 0 "U?" H 2150 4050 40  0000 C CNN
+F 0 "U2" H 2150 4050 40  0000 C CNN
 F 1 "MCP3550-60-E/SN" H 2400 4000 40  0000 C CNN
 F 2 "SO8" H 2500 3700 30  0000 C CIN
@@
 	1050 3700 2200 3700
 $Comp
-L MCP3550-60-E/SN U?
+L MCP3550-60-E/SN U3
 U 1 1 52F32ED6
 P 6500 6300
-F 0 "U?" H 5950 6650 40  0000 C CNN
+F 0 "U3" H 5950 6650 40  0000 C CNN
 F 1 "MCP3550-60-E/SN" H 6200 6600 40  0000 C CNN
 F 2 "SO8" H 6300 6300 30  0000 C CIN
@@
 $EndComp
 $Comp
-L ZENER D?
+L ZENER D3
 U 1 1 52F32EE3
 P 10400 6300
-F 0 "D?" H 10400 6400 50  0000 C CNN
+F 0 "D3" H 10400 6400 50  0000 C CNN
 F 1 "ZENER" H 10400 6200 40  0000 C CNN
 F 2 "~" H 10400 6300 60  0000 C CNN
@@
 $EndComp
 $Comp
-L +12V #PWR?
+L +12V #PWR08
 U 1 1 52F32EFC
 P 10400 5750
-F 0 "#PWR?" H 10400 5700 20  0001 C CNN
+F 0 "#PWR08" H 10400 5700 20  0001 C CNN
 F 1 "+12V" H 10400 5850 30  0000 C CNN
 F 2 "" H 10400 5750 60  0000 C CNN
@@
 Connection ~ 7800 6150
 $Comp
-L AGND #PWR?
+L AGND #PWR09
 U 1 1 52F33081
 P 7150 6600
-F 0 "#PWR?" H 7150 6600 40  0001 C CNN
+F 0 "#PWR09" H 7150 6600 40  0001 C CNN
 F 1 "AGND" H 7150 6530 50  0000 C CNN
 F 2 "" H 7150 6600 60  0000 C CNN
@@
 16-24 Bit ADC
 $Comp
-L AGND #PWR?
+L AGND #PWR010
 U 1 1 5302CE9A
 P 10400 6600
-F 0 "#PWR?" H 10400 6600 40  0001 C CNN
+F 0 "#PWR010" H 10400 6600 40  0001 C CNN
 F 1 "AGND" H 10400 6530 50  0000 C CNN
 F 2 "" H 10400 6600 60  0000 C CNN

Commit message: Thermocouple association and placement
Parts:
- removed D3: ZENER, ~, symbol ZENER
- removed U2, U3: MCP3550-60-E/SN, SO8, symbol MCP3550-60-E/SN
- removed unit 2 of U4
- added C10, C11, C7, C8, C9: C, ~, symbol C
- added P2: CONN_3X2, symbol CONN_3X2
- added P3: CONN_2, symbol CONN_2
- added R44, R45, R48, R49: R, ~, symbol R
- added U2: MCP3901, symbol MCP3901
- added U3: LMT84, symbol LMT84
- U4: value LM324 -> OPA4170
Connections:
- net labels added: +5V, CH0+, CH0-, CH1+, CH1-, REF+, REF-, ~CS, ~DR, ~RESET
- net labels removed: CS_N
- wire segments 45 -> 94
Other:
- note added: "TEMP SENSOR"
- note removed: "General Temperature Sensor"
- moved on the sheet: C1, R10, R11, R12, R13, R7, R8, R9, U4A, U4C, U4D
